File: Mini/OpenShock.kicad_pcb (KiCad board)
At the start: 2 copper layers, 58.8 x 46.2 mm, 42 parts, among them J1 USB_C_Receptacle_USB2.0, J2 Conn_01x03, J3 Conn_01x03, J4 Conn_01x06, J6 Conn_01x04, SW1 KH-6X6X6H-TJ, SW2 KH-6X6X6H-TJ, SW3 KH-6X6X6H-TJ, U1 ESP32-S3-WROOM-1, U2 AMS1117-3.3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

Commit message: Update rear silkscreen
Parts:
- added REF**: OSHW-Symbol_6.7x6mm_SilkScreen, Symbol:OSHW-Symbol_6.7x6mm_SilkScreen, B.Cu at (116.6, 94.0)
Other:
- board text added: "BASED ON NULLSTALGIA'S OPENSHOCK CORE V1.2"
- board text added: "github.com/comradef191/OpenShockMini"
- board text added: "r1.0"
- board text removed: "BASED ON NULLSTALGIA'S OPENSHOCK CORE V1.1"
- board text removed: "BIGASSGITHUBLINKHERE"

Commit message: Finalisation of PCB files
Parts:
- moved J1 0.49 mm to (70.0, 88.9)
Routing:
- net Net-(J1-SHIELD): track 36.5 -> 35.6 mm

Commit message: R1.1; Upgrade from AMS1117 to Low-Noise TI chip; TPS7A2033PDBVR, 300mA output
Added locally saved images of board, rather than Github cache.
Parts:
- removed C12: 22uF, Capacitor_SMD:C_0603_1608Metric_Pad1.08x0.95mm_HandSolder
- removed the C3 at (121.9, 92.8)
- removed the C4 at (121.9, 90.9)
- removed U3: MCP1700x-300xxTT, Package_TO_SOT_SMD:SOT-23_Handsoldering
- added C1: 1uF, Capacitor_SMD:C_0603_1608Metric_Pad1.08x0.95mm_HandSolder, F.Cu at (120.6, 85.2)
- added C10: 22uF, Capacitor_SMD:C_0603_1608Metric_Pad1.08x0.95mm_HandSolder, F.Cu at (120.6, 87.2)
- C2: renamed from C1; value 100nF -> 1uF
- C3: renamed from C2; value 10uF -> 22uF
- U2: value AMS1117-3.3 -> TPS7A2033PDBVR; footprint Package_TO_SOT_SMD:SOT-223-3_TabPin2 -> PCM_Package_TO_SOT_SMD_AKL:SOT-23-5_HandSoldering
- moved U2 1.39 mm to (115.6, 87.1)
- moved C11 1.34 mm to (120.6, 89.1)
- renumbered REF** to #SYM1, REF** to #SYM2, C10 to C4
Connections:
- U2 pad 1: GND -> +5V
- U2 pad 2: +3V3 -> GND
Routing:
- net +3V3: track 194.0 -> 176.1 mm
- net +5V: track 33.3 -> 31.5 mm
Other:
- board text added: "1uF"
- board text added: "5V->3V3"
- board text added: "REV 1.1"
- board text added: "r1.1"
- board text removed: "5V -> 3V3"
- board text removed: "REV 1.0"
- board text removed: "r1.0"

Commit message: r1.2; Board reshuffled for ease of add-on design, plus ESP32 soldering
Parts:
- moved J2 20.6 mm to (78.2, 82.3), turned to -90 degrees
- moved R2 13.7 mm to (73.3, 60.0), turned to 0 degrees
- moved J3 10.1 mm to (78.2, 76.7), turned to -90 degrees
- moved R9 9.84 mm to (73.3, 62.7), turned to 0 degrees
- moved U4 8.72 mm to (82.8, 69.7)
Connections:
- U1 pad 41: GND -> (no net)
Routing:
- net +3V3: track 176.1 -> 197.4 mm
- net /ANT.: track 22.6 -> 17.1 mm
- net SIGNAL: track 34.9 -> 33.3 mm
- net EN: track 57.4 -> 58.6 mm
Other:
- board text added: "REV 1.2"
- board text added: "r1.2"
- board text removed: "REV 1.1"
- board text removed: "r1.1"

Commit message: New revision; Board fixes
Parts:
- added J5: Conn_01x02, Connector_PinHeader_2.54mm:PinHeader_1x02_P2.54mm_Vertical, F.Cu at (126.9, 78.9)
- moved #SYM2 10.8 mm to (105.9, 93.0)
Connections:
- R7 pad 1: Net-(D4-A) -> Net-(J5-Pin_2)
- U1 pad 41: (no net) -> GND
Routing:
- net +3V3: track 197.4 -> 203.3 mm
- net Net-(J5-Pin_2): track 0.00 -> 3.80 mm
- net Net-(D4-A): track 14.6 -> 15.6 mm
- net SIGNAL: track 33.3 -> 32.6 mm
Other:
- board text added: "BASED ON NULLSTALGIA'S OPENSHOCK CORE V1.32"
- board text added: "BOOT"
- board text added: "CASE"
- board text added: "CC1"
- board text added: "CC2"
- board text added: "DEBUG"
- board text added: "DESIGNED BY PERA 7TH JULY, 2024"
- board text added: "RESET"
- board text added: "REV 1.3"
- board text added: "r1.3"
- board text removed: "100uF"
- board text removed: "BASED ON NULLSTALGIA'S OPENSHOCK CORE V1.2"
- board text removed: "DESIGNED BY PERA 21ST JUNE, 2024"
- board text removed: "REV 1.2"
- board text removed: "r1.2"

Commit message: New Revision.
Parts:
- removed C11, C3: 22uF, Capacitor_SMD:C_0603_1608Metric_Pad1.08x0.95mm_HandSolder
- added CN1: PJ-3200, EASYEDA Footprints:AUDIO-TH_PJ-3200, F.Cu at (126.0, 55.6)
- added H3: MountingHole, MountingHole:MountingHole_3.2mm_M3_ISO7380, F.Cu at (126.1, 91.9)
- added JP1: SolderJumper_2_Open, Jumper:SolderJumper-2_P1.3mm_Bridged_RoundedPad1.0x1.5mm, B.Cu at (125.0, 62.0)
- added JP2: SolderJumper_2_Open, Jumper:SolderJumper-2_P1.3mm_Bridged_RoundedPad1.0x1.5mm, B.Cu at (127.5, 62.0)
- added TP1: TestPoint, TestPoint:TestPoint_Pad_D1.5mm, B.Cu at (121.5, 89.9)
- added TP2: TestPoint, TestPoint:TestPoint_Pad_D1.5mm, B.Cu at (124.0, 87.4)
- added TP3: TestPoint, TestPoint:TestPoint_Pad_D1.5mm, B.Cu at (124.0, 84.9)
- added TP4: TestPoint, TestPoint:TestPoint_Pad_D1.5mm, B.Cu at (95.5, 84.9)
- added TP5: TestPoint, TestPoint:TestPoint_Pad_D1.5mm, B.Cu at (95.5, 87.8)
- added TP6: TestPoint, TestPoint:TestPoint_Pad_D1.5mm, B.Cu at (101.1, 84.9)
- added TP7: TestPoint, TestPoint:TestPoint_Pad_D1.5mm, B.Cu at (101.1, 87.8)
- added TP8: TestPoint, TestPoint:TestPoint_Pad_D1.5mm, B.Cu at (101.1, 90.6)
- added TP9: TestPoint, TestPoint:TestPoint_Pad_D1.5mm, B.Cu at (95.5, 90.6)
- C1, C10, C2, C4, C5, C6, C7, C8, C9: footprint Capacitor_SMD:C_0603_1608Metric_Pad1.08x0.95mm_HandSolder -> Capacitor_SMD:C_0805_2012Metric_Pad1.18x1.45mm_HandSolder
- J5: value Conn_01x02 -> USB_B_Mini; footprint Connector_PinHeader_2.54mm:PinHeader_1x02_P2.54mm_Vertical -> EASYEDA Footprints:MICRO-USB-TH_UX-150-ARG4
- R6: value 5.1k -> 10k
- U1: footprint RF_Module:ESP32-S3-WROOM-1 -> CustomFootprints:ESP32-S3-WROOM-1
- U2: value TPS7A2033PDBVR -> AMS1117-3.3; footprint PCM_Package_TO_SOT_SMD_AKL:SOT-23-5_HandSoldering -> Package_TO_SOT_SMD:SOT-89-3_Handsoldering
- moved J5 51.1 mm to (75.8, 79.6), turned to -90 degrees
- moved C7 12.5 mm to (123.9, 65.2), turned to 90 degrees
- moved J2 8.40 mm to (86.6, 82.5)
- moved J3 8.40 mm to (86.6, 76.9)
- moved D1 7.52 mm to (127.5, 66.0)
- moved D4 6.28 mm to (127.5, 74.3)
- moved D3 5.04 mm to (127.5, 80.5)
- moved AE1 1.52 mm to (82.3, 53.8), turned to 90 degrees
- moved R6 1.27 mm to (122.8, 81.5)
- moved C4 1.26 mm to (110.7, 87.9)
- moved R7 1.24 mm to (122.8, 78.7)
- moved C6 1.19 mm to (74.7, 54.3)
- moved C5 1.19 mm to (74.7, 57.0)
- moved #SYM2 0.85 mm to (106.7, 93.0)
- moved C10 0.70 mm to (120.6, 87.9)
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Connections:
- net Net-(J1-CC1) renamed /CC1
- net Net-(J1-CC2) renamed /CC2
- J5 pad 1: Net-(D4-A) -> +5VA
- J5 pad 2: Net-(J5-Pin_2) -> D-
- R7 pad 1: Net-(J5-Pin_2) -> Net-(D4-A)
- U2 pad 1: +5V -> GND
- U2 pad 2: GND -> +3V3
Routing:
- net D-: track 51.5 -> 84.0 mm, vias 2 -> 4
- net D+: track 54.6 -> 84.7 mm, vias 2 -> 3
- net E_STOP: track 34.7 -> 52.4 mm, vias 1 -> 2
- net +5VA: track 38.0 -> 55.3 mm, vias 0 -> 2
- net Net-(J1-SHIELD): track 35.6 -> 49.8 mm
- net RGB: track 40.0 -> 52.2 mm
- net Net-(JP1-A): track 0.00 -> 9.41 mm
- net Net-(JP2-A): track 0.00 -> 7.58 mm
- net Net-(D4-A): track 15.6 -> 8.70 mm
- net +5V: track 31.5 -> 36.6 mm, vias 0 -> 1
- net +3V3: track 203.3 -> 199.2 mm, vias 2 -> 3
- net Net-(J5-Pin_2): track 3.80 -> 0.00 mm
- net Net-(D3-A): track 9.82 -> 6.15 mm
- net SIGNAL: track 32.6 -> 35.9 mm, vias 0 -> 1
- net /CC2: track 24.1 -> 26.4 mm
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Other:
- board text added: "15SEP24"
- board text added: "ADD ONLY ONE USB CONNECTOR"
- board text added: "AMS1117"
- board text added: "ANTENNA"
- board text added: "BASED ON NULLSTALGIA'S OPENSHOCK CORE V1.2"
- board text added: "DESIGNED BY"
- board text added: "ESTOP CONN."
- board text added: "Fill this last!"
- board text added: "ONLY NEEDED WITH USB-C"
- board text added: "TRANSMITTER"
- board text added: "USB Mini B"
- board text added: "USB-C"
- board text added: "VIN"
- board text added: "[PERA]"
- board text added: "ijo[pilin=epiku=wawa=anpa=]"
- board text removed: "433MHz ANTENNA"
- board text removed: "BASED ON NULLSTALGIA'S OPENSHOCK CORE V1.32"
- board text removed: "CASE"
- board text removed: "DESIGNED BY PERA 7TH JULY, 2024"
- board text removed: "ESP32-S3 WROOM-1"
- board text removed: "god, i hate USB-C"
